File: schematics/camera_pelican.kicad_sch (KiCad schematic)
At the start: 7 parts, among them J4 0.5K-A-20PB, Q5 NDS7002A

Commit message: updated schematic based on review
Parts:
- added C402: 100nF, C_GRM155R71C104KA88D:C_GRM155R71C104KA88D, symbol C_GRM155R71C104KA88D:GRM155R71C104KA88D
- renumbered C18 to C401, LED2 to CAM_LED401, J4 to MIPI_J401, Q5 to Q401, R27 to R401, R28 to R402, R20 to R403
Connections:
- net GND: now also C402.2
- net VCC_3V3: now also C402.1
Other:
- moved on the sheet: C401, CAM_LED401, MIPI_J401, Q401, R401, R402, R403
