File: schematics/power_pelican.kicad_sch (KiCad schematic)
At the start: 43 parts, among them J1 436500200, J2 436500200, Q1 DMG2305UX-13, Q2 DMG2305UX-13, Q3 NDS7002A, Q4 NDS7002A, U1 TPS61023DRLR, U2 TPS2116DRLR, U3 BQ24074RGTT

Commit message: updated schematic based on review
Parts:
- renumbered J1 to BAT_J201, LED1 to BAT_LED201, U1 to BOOST_U202, C7 to C201, C8 to C202, C9 to C203, C10 to C204, C11 to C205, C12 to C206, C1 to C207, C2 to C208, C3 to C209, C4 to C210, C6 to C211, C5 to C212, U3 to CHG_U203, L1 to L201, U2 to MUX_U201, Q4 to Q201, Q2 to Q202, Q1 to Q203, Q3 to Q204, R17 to R201, R7 to R202, R32 to R203, R8 to R204, R34 to R205, R14 to R206, R15 to R207, R16 to R208, R4 to R209, R5 to R210, R6 to R211, R1 to R212, R2 to R213, R3 to R214, R11 to R215, R9 to R216, R12 to R217, R35 to R218, R13 to R219, R10 to R220, J2 to SW_J202
Connections:
- net VCC_5V0: no longer C210.1, CHG_U203.13 (IN)
- net VUSB: now also C210.1, CHG_U203.13 (IN)
- net SWITCH_STAT renamed SW_STAT
Other:
- note added: "Boost Converter"
- note removed: "Power Regulation"
