File: schematics/storage_pelican.kicad_sch (KiCad schematic)
At the start: 5 parts, among them J3 TF-115-BCP9

Commit message: updated schematic based on review
Parts:
- renumbered C13 to C601, R31 to R601, R21 to R602, LED9 to STORE_LED601, J3 to uSD_J601
Connections:
- net LED_STOR renamed LED_STORE
Changed lines of the file:
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@@
 		)
 	)
-	(global_label "LED_STOR"
+	(global_label "LED_STORE"
 		(shape input)
 		(at 90.17 90.17 180)
@@
 		)
 		(property "Intersheetrefs" "${INTERSHEET_REFS}"
-			(at 77.9925 90.17 0)
+			(at 76.8435 90.17 0)
 			(hide yes)
 			(show_name no)
@@
 		(in_pos_files yes)
 		(dnp no)
-		(property "Reference" "C13"
+		(property "Reference" "C601"
 			(at 90.932 63.5 90)
 			(show_name no)
@@
 			(project "pelican"
 				(path "/03ccc822-2fac-4029-af97-539e9460fe35/a85a53bb-5b50-475b-995a-b454556c96ce"
-					(reference "C13")
+					(reference "C601")
 					(unit 1)
 				)
@@
 		(in_pos_files yes)
 		(dnp no)
-		(property "Reference" "R31"
+		(property "Reference" "R601"
 			(at 76.2 63.4999 90)
 			(show_name no)
@@
 			(project "pelican"
 				(path "/03ccc822-2fac-4029-af97-539e9460fe35/a85a53bb-5b50-475b-995a-b454556c96ce"
-					(reference "R31")
+					(reference "R601")
 					(unit 1)
 				)
@@
 		(dnp no)
 		(fields_autoplaced yes)
-		(property "Reference" "#PWR95"
+		(property "Reference" "#PWR0605"
 			(at 100.33 74.93 0)
 			(hide yes)
@@
 			(project "pelican"
 				(path "/03ccc822-2fac-4029-af97-539e9460fe35/a85a53bb-5b50-475b-995a-b454556c96ce"
-					(reference "#PWR95")
+					(reference "#PWR0605")
 					(unit 1)
 				)
@@
 		(dnp no)
 		(fields_autoplaced yes)
-		(property "Reference" "LED9"
+		(property "Reference" "STORE_LED601"
 			(at 115.06 83.82 0)
 			(show_name no)
@@
 			(project "pelican"
 				(path "/03ccc822-2fac-4029-af97-539e9460fe35/a85a53bb-5b50-475b-995a-b454556c96ce"
-					(reference "LED9")
+					(reference "STORE_LED601")
 					(unit 1)
 				)
@@
 		(dnp no)
 		(fields_autoplaced yes)
-		(property "Reference" "#PWR66"
+		(property "Reference" "#PWR0606"
 			(at 123.19 96.52 0)
 			(hide yes)
@@
 			(project "pelican"
 				(path "/03ccc822-2fac-4029-af97-539e9460fe35/a85a53bb-5b50-475b-995a-b454556c96ce"
-					(reference "#PWR66")
+					(reference "#PWR0606")
 					(unit 1)
 				)
@@
 		(dnp no)
 		(fields_autoplaced yes)
-		(property "Reference" "R21"
+		(property "Reference" "R602"
 			(at 99.06 83.82 0)
 			(show_name no)
@@
 			(project "pelican"
 				(path "/03ccc822-2fac-4029-af97-539e9460fe35/a85a53bb-5b50-475b-995a-b454556c96ce"
-					(reference "R21")
+					(reference "R602")
 					(unit 1)
 				)
@@
 		(in_pos_files yes)
 		(dnp no)
-		(property "Reference" "#PWR96"
+		(property "Reference" "#PWR0604"
 			(at 100.33 50.8 0)
 			(hide yes)
@@
 			(project "pelican"
 				(path "/03ccc822-2fac-4029-af97-539e9460fe35/a85a53bb-5b50-475b-995a-b454556c96ce"
-					(reference "#PWR96")
+					(reference "#PWR0604")
 					(unit 1)
 				)
@@
 		(in_pos_files yes)
 		(dnp no)
-		(property "Reference" "#PWR97"
+		(property "Reference" "#PWR0603"
 			(at 100.33 43.18 0)
 			(hide yes)
@@
 			(project "pelican"
 				(path "/03ccc822-2fac-4029-af97-539e9460fe35/a85a53bb-5b50-475b-995a-b454556c96ce"
-					(reference "#PWR97")
+					(reference "#PWR0603")
 					(unit 1)
 				)
@@
 		(dnp no)
 		(fields_autoplaced yes)
-		(property "Reference" "J3"
+		(property "Reference" "uSD_J601"
 			(at 134.62 45.7199 0)
 			(show_name no)
@@
 			(project "pelican"
 				(path "/03ccc822-2fac-4029-af97-539e9460fe35/a85a53bb-5b50-475b-995a-b454556c96ce"
-					(reference "J3")
+					(reference "uSD_J601")
 					(unit 1)
 				)
@@
 		(in_pos_files yes)
 		(dnp no)
-		(property "Reference" "#PWR94"
+		(property "Reference" "#PWR0601"
 			(at 66.04 74.93 0)
 			(hide yes)
@@
 			(project "pelican"
 				(path "/03ccc822-2fac-4029-af97-539e9460fe35/a85a53bb-5b50-475b-995a-b454556c96ce"
-					(reference "#PWR94")
+					(reference "#PWR0601")
 					(unit 1)
 				)
@@
 		(in_pos_files yes)
 		(dnp no)
-		(property "Reference" "#PWR55"
+		(property "Reference" "#PWR0602"
 			(at 93.98 64.77 0)
 			(hide yes)
@@
 			(project "pelican"
 				(path "/03ccc822-2fac-4029-af97-539e9460fe35/a85a53bb-5b50-475b-995a-b454556c96ce"
-					(reference "#PWR55")
+					(reference "#PWR0602")
 					(unit 1)
 				)
