File: schematics/usb_pelican.kicad_sch (KiCad schematic)
At the start: 6 parts, among them J7 USB-C-16P

Commit message: updated schematic based on review
Parts:
- added C701: 100nF, C_GRM155R71C104KA88D:C_GRM155R71C104KA88D, symbol C_GRM155R71C104KA88D:GRM155R71C104KA88D
- renumbered D1 to ESD_D701, R22 to R701, R30 to R702, R33 to R703, R18 to R704, J7 to USBC_J701
Connections:
- net GND: now also C701.2; no longer R701.1, R702.1, USBC_J701.1 (GND1), USBC_J701.13 (SHIELD1), USBC_J701.14 (SHIELD2), USBC_J701.2 (GND2)
- new net GNDUSB: C701.1, R701.1, R702.1, USBC_J701.1 (GND1), USBC_J701.13 (SHIELD1), USBC_J701.14 (SHIELD2), USBC_J701.2 (GND2)
Other:
- moved on the sheet: ESD_D701, R701, R702, R703, R704, USBC_J701
