File: pelican/schematics/camera_pelican.kicad_sch (KiCad schematic)
At the start: 8 parts, among them Q401 NDS7002A

Commit message: Update Pelican design libraries and save connector layout concept
Parts:
- C401, C402: LCSC Part # C71629 -> C1525
- CAM_LED401: value LTST-C193KRKT-5A -> KT-0603R; LCSC Part # C157741 -> C2286
- R401, R402: LCSC Part # C105871 -> C25900
- R403: value 100R -> 200R; LCSC Part # C106232 -> C25087
Connections:
- net CAM_RESET renamed CAM_RST_N
Changed lines of the file:
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@@
 		)
 	)
-	(label "CAM_RESET"
+	(label "CAM_RST_N"
 		(at 86.36 63.5 0)
 		(effects
@@
 			)
 		)
-		(property "LCSC Part #" "C71629"
+		(property "LCSC Part #" "C1525"
 			(at 86.36 73.66 0)
 			(hide yes)
@@
 			)
 		)
-		(property "LCSC Part #" "C105871"
+		(property "LCSC Part #" "C25900"
 			(at 36.83 46.99 0)
 			(hide yes)
@@
 			)
 		)
-		(property "Value" "100R"
+		(property "Value" "200R"
 			(at 149.86 46.9899 90)
 			(show_name no)
@@
 			)
 		)
-		(property "LCSC Part #" "C106232"
+		(property "LCSC Part #" "C25087"
 			(at 147.32 39.37 0)
 			(hide yes)
@@
 			)
 		)
-		(property "Value" "LTST-C193KRKT-5A"
+		(property "Value" "KT-0603R"
 			(at 153.67 62.2299 90)
 			(show_name no)
@@
 			)
 		)
-		(property "LCSC Part #" "C157741"
+		(property "LCSC Part #" "C2286"
 			(at 147.32 54.61 0)
 			(hide yes)
@@
 			)
 		)
-		(property "LCSC Part #" "C71629"
+		(property "LCSC Part #" "C1525"
 			(at 71.12 73.66 0)
 			(hide yes)
@@
 			)
 		)
-		(property "LCSC Part #" "C105871"
+		(property "LCSC Part #" "C25900"
 			(at 123.19 48.26 0)
 			(hide yes)
