File: pelican/schematics/core_pelican.kicad_sch (KiCad schematic)
At the start: 16 parts

Commit message: Update Pelican design libraries and save connector layout concept
Parts:
- removed DEBUG_LED303: SZYY0402YG, LED_SZYY0402YG:LED_SZYY0402YG, symbol LED_SZYY0402YG:SZYY0402YG
- removed R303: 10K, R_RC0402FR:R_RC0402FR, symbol R_RC0402FR:RC0402FR-0710KL
- removed UART_J301: 61300411121, J_61300411121:J_61300411121, symbol J_61300411121:61300411121
- added UART_TP303, UART_TP304, UART_TP305, UART_TP306: TestPoint, testpoint:TestPoint_Pad_D1.5mm, symbol testpoint:TestPoint
- C301, C302: LCSC Part # C71629 -> C1525
- JTAG_TP301, JTAG_TP302: footprint (none) -> testpoint:TestPoint_Pad_D1.5mm
- R301, R302, R304, R305: LCSC Part # C60490 -> C25744
Connections:
- net MIC0_N is gone; now on net GND: SOC_U301.32 (CODEC_MIC0N)
- net GND: now also UART_TP306.1
- net LED_ALIVE: now also SOC_U301.97 (VO_LCDC_D3/VI_CIF_D6_M1/PWM8_M1/UART4_RX_M1/SDIO_D3_M1/GPIO1_C4_d); no longer SOC_U301.101 (VO_LCDC_D7/VI_CIF_D2_M1/PWM2_M2/SPI0_CS0_M0/SDIO_D1_M1/GPIO1_C0_d)
- net LED_BAT: now also SOC_U301.95 (VO_LCDC_D1/VI_CIF_D8_M1/PWM10_M1/UART4_RTS_M1/GPIO1_C6_d); no longer SOC_U301.98 (VO_LCDC_D4/VI_CIF_D5_M1/PWM6_M2/I2C4_SDA_M1/SDIO_CMD_M1/SPI0_MISO_M0/GPIO1_C3_d)
- net LED_ETH_GREEN: now also SOC_U301.93 (VO_LCDC_DEN/VI_CIF_CLKI_M1/PWM3_IR_M2/UART5_RTS_M1/UART3_TX_M1/GPIO1_D0_d); no longer SOC_U301.95 (VO_LCDC_D1/VI_CIF_D8_M1/PWM10_M1/UART4_RTS_M1/GPIO1_C6_d)
- net LED_ETH_YELLOW: now also SOC_U301.92 (VO_LCDC_HSYNC/VI_CIF_HREF_M1/PWM10_M2/UART5_CTS_M1/UART3_RX_M1/GPIO1_D1_d); no longer SOC_U301.94 (VO_LCDC_D0/VI_CIF_D9_M1/PWM11_IR_M1/UART4_CTS_M1/GPIO1_C7_d)
- net LED_REC: now also SOC_U301.94 (VO_LCDC_D0/VI_CIF_D9_M1/PWM11_IR_M1/UART4_CTS_M1/GPIO1_C7_d); no longer SOC_U301.97 (VO_LCDC_D3/VI_CIF_D6_M1/PWM8_M1/UART4_RX_M1/SDIO_D3_M1/GPIO1_C4_d)
- net UART_RX: now also UART_TP305.1
- net UART_TX: now also UART_TP304.1
- net VCC_3V3: now also UART_TP303.1
- net BAT_CHG_SRC_STAT renamed CHG_IN_VLD_N
- net BAT_CHG_STAT renamed CHG_STAT_N
- net BAT_V_STAT renamed VBAT_SNS
- net CAM_RESET renamed CAM_RST_N
- net HOLD_PWR renamed PWR_HOLD
- net LED_DEBUG renamed LED_HEALTH
- net LED_HEALTH: now also R302.2
- net LED_STORE: no longer names the net of SOC_U301.99 (VO_LCDC_D5/VI_CIF_D4_M1/PWM5_M2/I2C4_SCL_M1/SDIO_CLK_M1/SPI0_MOSI_M0/GPIO1_C2_d)
- net LED_UART: no longer names the net of SOC_U301.100 (VO_LCDC_D6/VI_CIF_D3_M1/PWM4_M2/SPI0_CLK_M0/SDIO_D0_M1/GPIO1_C1_d)
- net LED_UART: no longer R302.2
- net PWR_SRC renamed PWR_SRC_STAT
- no-connect marks 44 -> 46
