File: pelican/schematics/ethernet_pelican.kicad_sch (KiCad schematic)
At the start: 7 parts

Commit message: Update Pelican design libraries and save connector layout concept
Parts:
- removed ETH_J801: RJ45-HANRUN, J_RJ45-HANRUN:J_RJ45-HANRUN_TH, symbol J_RJ45-HANRUN:RJ45-HANRUN
- added J801: HR911105A, J_HR911105A:J_HR911105A_TH, symbol J_HR911105A:HR911105A
- C801, C804: LCSC Part C318577 -> C15195; LCSC Part # C318577 -> C15195
- C802: LCSC Part # C71629 -> C1525
- R801, R802: LCSC Part # (none) -> C25087
Connections:
- net CT_RX: now also J801.5 (CT_RX)
- net CT_TX: now also J801.4 (CT_TX)
- net ETH_RX_N: now also J801.6 (RD-)
- net ETH_RX_P: now also J801.3 (RD+)
- net ETH_TX_N: now also J801.2 (TD-)
- net ETH_TX_P: now also J801.1 (TD+)
- net GND: now also J801.10 (LED1-), J801.11 (LED2-)
- net GNDETH: now also J801.8 (CHSGND), J801.SH1 (SHIELD), J801.SH2 (SHIELD)
- net at R802.1: now also J801.12 (LED2+)
- net at R801.1: now also J801.9 (LED1+)
Changed lines of the file:
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@@
 			)
 		)
-		(property "LCSC Part #" "C318577"
+		(property "LCSC Part #" "C15195"
 			(at 58.42 49.53 0)
 			(hide yes)
@@
 			)
 		)
-		(property "LCSC Part" "C318577"
+		(property "LCSC Part" "C15195"
 			(at 58.42 49.53 0)
 			(hide yes)
@@
 				(path "/03ccc822-2fac-4029-af97-539e9460fe35/21ae68ba-843b-4af3-805b-206ec5f29f16"
 					(reference "C801")
-					(unit 1)
-				)
-			)
-		)
-	)
-	(symbol
-		(lib_id "J_RJ45-HANRUN:RJ45-HANRUN")
-		(at 142.24 55.88 0)
-		(unit 1)
-		(body_style 1)
-		(exclude_from_sim no)
-		(in_bom yes)
-		(on_board yes)
-		(in_pos_files yes)
-		(dnp no)
-		(fields_autoplaced yes)
-		(property "Reference" "ETH_J801"
-			(at 156.21 52.0699 0)
-			(show_name no)
-			(do_not_autoplace no)
-			(effects
-				(font
-					(size 1.27 1.27)
-				)
-				(justify left)
-			)
-		)
-		(property "Value" "RJ45-HANRUN"
-			(at 156.21 54.6099 0)
-			(show_name no)
-			(do_not_autoplace no)
-			(effects
-				(font
-					(size 1.27 1.27)
-				)
-				(justify left)
-			)
-		)
-		(property "Footprint" "J_RJ45-HANRUN:J_RJ45-HANRUN_TH"
-			(at 142.24 83.82 0)
-			(hide yes)
-			(show_name no)
-			(do_not_autoplace no)
-			(effects
-				(font
-					(size 1.27 1.27)
-				)
-			)
-		)
-		(property "Datasheet" "https://lcsc.com/product-detail/Ethernet-Connectors-Modular-Connectors_Zhongshan-HanRun-Elec-HY951180A_C34677.html"
-			(at 142.24 86.36 0)
-			(hide yes)
-			(show_name no)
-			(do_not_autoplace no)
-			(effects
-				(font
-					(size 1.27 1.27)
-				)
-			)
-		)
-		(property "Description" "RJ45 Ethernet jack with integrated magnetics and status LEDs. One shared symbol, two mount-style footprints: J_RJ45-HANRUN_TH (through hole, HY951180A/C34677, default) and J_RJ45-HANRUN_SMD (surface mount, HR961160C/C55683). Pin numbers are canonical across both footprints (SMD footprint pads were renumbered from the vendor's native numbering to match). When placing the SMD variant, override this instance's Footprint/MPN/LCSC Part/Datasheet fields to the _SMD values."
-			(at 142.24 55.88 0)
-			(hide yes)
-			(show_name no)
-			(do_not_autoplace no)
-			(effects
-				(font
-					(size 1.27 1.27)
-				)
-			)
-		)
-		(property "LCSC Part #" "C34677"
-			(at 142.24 86.36 0)
-			(hide yes)
-			(show_name no)
-			(do_not_autoplace no)
-			(effects
-				(font
-					(size 1.27 1.27)
-				)
-			)
-		)
-		(property "Manufacturer" "HANRUN(Zhongshan HanRun Elec)"
-			(at 142.24 88.9 0)
-			(hide yes)
-			(show_name no)
-			(do_not_autoplace no)
-			(effects
-				(font
-					(size 1.27 1.27)
-				)
-			)
-		)
-		(property "MPN" "HY951180A"
-			(at 142.24 91.44 0)
-			(hide yes)
-			(show_name no)
-			(do_not_autoplace no)
-			(effects
-				(font
-					(size 1.27 1.27)
-				)
-			)
-		)
-		(property "LCSC Part" "C34677"
-			(at 142.24 93.98 0)
-			(hide yes)
-			(show_name no)
-			(do_not_autoplace no)
-			(effects
-				(font
-					(size 1.27 1.27)
-				)
-			)
-		)
-		(property "MPN_SMD" "HR961160C"
-			(at 142.24 96.52 0)
-			(hide yes)
-			(show_name no)
-			(do_not_autoplace no)
-			(effects
-				(font
-					(size 1.27 1.27)
-				)
-			)
-		)
-		(property "LCSC Part_SMD" "C55683"
-			(at 142.24 99.06 0)
-			(hide yes)
-			(show_name no)
-			(do_not_autoplace no)
-			(effects
-				(font
-					(size 1.27 1.27)
-				)
-			)
-		)
-		(property "Datasheet_SMD" "https://lcsc.com/product-detail/Ethernet-Connectors-Modular-Connectors_Zhongshan-HanRun-Elec-HR961160C_C55683.html"
-			(at 142.24 101.6 0)
-			(hide yes)
-			(show_name no)
-			(do_not_autoplace no)
-			(effects
-				(font
-					(size 1.27 1.27)
-				)
-			)
-		)
-		(pin "1"
-		)
-		(pin "3"
-		)
-		(pin "4"
-		)
-		(pin "5"
-		)
-		(pin "6"
-		)
-		(pin "7"
-		)
-		(pin "8"
-		)
-		(pin "9"
-		)
-		(pin "10"
-		)
-		(pin "11"
-		)
-		(pin "12"
-		)
-		(pin "13"
-		)
-		(pin "14"
-		)
-		(pin "2"
-		)
-		(instances
-			(project "pelican"
-				(path "/03ccc822-2fac-4029-af97-539e9460fe35/21ae68ba-843b-4af3-805b-206ec5f29f16"
-					(reference "ETH_J801")
 					(unit 1)
 				)
@@
 			)
 		)
+		(property "LCSC Part #" "C25087"
+			(at 104.14 63.5 0)
+			(hide yes)
+			(show_name no)
+			(do_not_autoplace no)
+			(effects
+				(font
+					(size 1.27 1.27)
+				)
+			)
+		)
 		(pin "1"
 		)
@@
 			)
 		)
-		(property "LCSC Part #" "C71629"
+		(property "LCSC Part #" "C1525"
 			(at 58.42 67.31 0)
 			(hide yes)
@@
 	)
 	(symbol
+		(lib_id "J_HR911105A:HR911105A")
+		(at 142.24 55.88 0)
+		(unit 1)
+		(body_style 1)
+		(exclude_from_sim no)
+		(in_bom yes)
+		(on_board yes)
+		(in_pos_files yes)
+		(dnp no)
+		(fields_autoplaced yes)
+		(property "Reference" "J801"
+			(at 156.21 52.0699 0)
+			(show_name no)
+			(do_not_autoplace no)
+			(effects
+				(font
+					(size 1.27 1.27)
+				)
+				(justify left)
+			)
+		)
+		(property "Value" "HR911105A"
+			(at 156.21 54.6099 0)
+			(show_name no)
+			(do_not_autoplace no)
+			(effects
+				(font
+					(size 1.27 1.27)
+				)
+				(justify left)
+			)
+		)
+		(property "Footprint" "J_HR911105A:J_HR911105A_TH"
+			(at 142.24 83.82 0)
+			(hide yes)
+			(show_name no)
+			(do_not_autoplace no)
+			(effects
+				(font
+					(size 1.27 1.27)
+				)
+			)
+		)
+		(property "Datasheet" "https://lcsc.com/product-detail/RJ45_RJ45-LED_C12074.html"
+			(at 142.24 86.36 0)
+			(hide yes)
+			(show_name no)
+			(do_not_autoplace no)
+			(effects
+				(font
+					(size 1.27 1.27)
+				)
+			)
+		)
+		(property "Description" "RJ45 Ethernet jack with integrated magnetics and status LEDs (HanRun HR911105A, LCSC C12074). Symbol redrawn to match the previous RJ45-HANRUN layout for drop-in rewiring; pin numbers map to the HR911105A_TH through-hole footprint (1-12 + SH1/SH2). Pins 4/5 are the TX/RX center taps; pins 7/8 are the magnetics termination / chassis pins - verify against the HR911105A datasheet before finalizing."
+			(at 142.24 55.88 0)
+			(hide yes)
+			(show_name no)
+			(do_not_autoplace no)
+			(effects
+				(font
+					(size 1.27 1.27)
+				)
+			)
+		)
+		(property "Manufacturer" "HANRUN(汉仁)"
+			(at 142.24 88.9 0)
+			(hide yes)
+			(show_name no)
+			(do_not_autoplace no)
+			(effects
+				(font
+					(size 1.27 1.27)
+				)
+			)
+		)
+		(property "MPN" "HR911105A"
+			(at 142.24 91.44 0)
+			(hide yes)
+			(show_name no)
+			(do_not_autoplace no)
+			(effects
+				(font
+					(size 1.27 1.27)
+				)
+			)
+		)
+		(property "LCSC Part" "C12074"
+			(at 142.24 93.98 0)
+			(hide yes)
+			(show_name no)
+			(do_not_autoplace no)
+			(effects
+				(font
+					(size 1.27 1.27)
+				)
+			)
+		)
+		(pin "8"
+		)
+		(pin "10"
+		)
+		(pin "9"
+		)
+		(pin "7"
+		)
+		(pin "11"
+		)
+		(pin "1"
+		)
+		(pin "SH1"
+		)
+		(pin "12"
+		)
+		(pin "SH2"
+		)
+		(pin "3"
+		)
+		(pin "4"
+		)
+		(pin "2"
+		)
+		(pin "5"
+		)
+		(pin "6"
+		)
+		(instances
+			(project "pelican"
+				(path "/03ccc822-2fac-4029-af97-539e9460fe35/21ae68ba-843b-4af3-805b-206ec5f29f16"
+					(reference "J801")
+					(unit 1)
+				)
+			)
+		)
+	)
+	(symbol
 		(lib_id "R_RC0402FR:RC0402FR-07200RL")
 		(at 104.14 77.47 0)
@@
 		)
 		(property "Description" ""
+			(at 104.14 77.47 0)
+			(hide yes)
+			(show_name no)
+			(do_not_autoplace no)
+			(effects
+				(font
+					(size 1.27 1.27)
+				)
+			)
+		)
+		(property "LCSC Part #" "C25087"
 			(at 104.14 77.47 0)
 			(hide yes)
@@
 			)
 		)
-		(property "LCSC Part #" "C318577"
+		(property "LCSC Part #" "C15195"
 			(at 66.04 55.88 0)
 			(hide yes)
@@
 			)
 		)
-		(property "LCSC Part" "C318577"
+		(property "LCSC Part" "C15195"
 			(at 66.04 55.88 0)
 			(hide yes)
