File: pelican/schematics/power_pelican.kicad_sch (KiCad schematic)
At the start: 43 parts, among them Q201 NDS7002A, Q202 DMG2305UX-13, Q203 DMG2305UX-13, Q204 NDS7002A

Commit message: Update Pelican design libraries and save connector layout concept
Parts:
- removed BAT_J201, SW_J202: 436500200, J_436500200:J_436500200, symbol J_436500200:436500200
- added CN201: 43045-0401, J_43045-0401:J_43045-0401_2x02_RA, symbol J_43045-0401:43045-0401
- BAT_LED201: value LTST-C193KGKT-5A -> APTD1608CGCK; LCSC Part # C125102 -> C5121471
- C203, C204, C206: LCSC Part # C71629 -> C1525
- C207, C211, C212: LCSC Part # C71633 -> C19666
- C210: LCSC Part # C76999 -> C52923
- R201: value 100K -> 10K; symbol R_RC0402FR:RC0402FR-07100KL -> R_RC0402FR:RC0402FR-0710KL; LCSC Part # C60490 -> C25744
- R202, R208: LCSC Part # C106232 -> C25076
- R203, R204, R205, R207, R210, R212, R214, R215: LCSC Part # C60491 -> C25741
- R206: LCSC Part # C114763 -> C25764
- R211, R218, R219, R220: LCSC Part # C60490 -> C25744
Connections:
- net GND: now also CN201.2, CN201.4
- net SW_STAT: now also CN201.3
- net VBAT: now also CN201.1
- net BAT_CHG_SRC_STAT renamed CHG_IN_VLD_N
- net BAT_CHG_STAT renamed CHG_STAT_N
- net BAT_V_STAT renamed VBAT_SNS
- net HOLD_PWR renamed PWR_HOLD
- net PWR_SRC renamed PWR_SRC_STAT
Other:
- moved on the sheet: BAT_LED201, Q201, Q202, Q203, Q204, R201, R202, R203, R204, R205, R206, R207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
