File: pelican/schematics/storage_pelican.kicad_sch (KiCad schematic)
At the start: 5 parts

Commit message: Update Pelican design libraries and save connector layout concept
Parts:
- removed R602: 10K, R_RC0402FR:R_RC0402FR, symbol R_RC0402FR:RC0402FR-0710KL
- removed STORE_LED601: SZYY0402YG, LED_SZYY0402YG:LED_SZYY0402YG, symbol LED_SZYY0402YG:SZYY0402YG
- C601: LCSC Part # C71629 -> C1525
- R601: LCSC Part # C60490 -> C25744
