File: Flamingo/flamingo.kicad_sch (KiCad schematic)
At the start: 0 parts

Commit message: adding last pages
Other:
- added sheet SD card (schematics\SD_card.kicad_sch)
Changed lines of the file:
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@@
 	)
 	(sheet
-		(at 63.5 52.07)
+		(at 74.93 54.61)
 		(size 55.88 25.4)
 		(exclude_from_sim no)
@@
 		)
 		(property "Sheetname" "Camera"
-			(at 63.5 51.3584 0)
+			(at 74.93 53.8984 0)
 			(show_name no)
 			(do_not_autoplace no)
@@
 		)
 		(property "Sheetfile" "schematics\\camera.kicad_sch"
-			(at 63.5 78.0546 0)
+			(at 74.93 80.5946 0)
 			(show_name no)
 			(do_not_autoplace no)
@@
 	(sheet
 		(at 20.32 102.87)
-		(size 86.36 10.16)
+		(size 110.49 12.7)
 		(exclude_from_sim no)
 		(in_bom yes)
@@
 		)
 		(property "Sheetfile" "schematics\\usb_debug.kicad_sch"
-			(at 20.32 113.6146 0)
+			(at 20.32 116.1546 0)
 			(show_name no)
 			(do_not_autoplace no)
@@
 	(sheet
 		(at 20.32 87.63)
-		(size 86.36 10.16)
+		(size 110.49 11.43)
 		(exclude_from_sim no)
 		(in_bom yes)
@@
 		)
 		(property "Sheetfile" "schematics\\usb_power_program.kicad_sch"
-			(at 20.32 98.3746 0)
+			(at 20.32 99.6446 0)
 			(show_name no)
 			(do_not_autoplace no)
@@
 	(sheet
 		(at 19.05 24.13)
-		(size 93.98 17.78)
+		(size 111.76 19.05)
 		(exclude_from_sim no)
 		(in_bom yes)
@@
 		)
 		(property "Sheetfile" "schematics\\power.kicad_sch"
-			(at 19.05 42.4946 0)
+			(at 19.05 43.7646 0)
 			(show_name no)
 			(do_not_autoplace no)
@@
 				)
 			)
+		)
+	)
+	(sheet
+		(at 20.32 143.51)
+		(size 110.49 12.7)
+		(exclude_from_sim no)
+		(in_bom yes)
+		(on_board yes)
+		(dnp no)
+		(fields_autoplaced yes)
+		(stroke
+			(width 0.1524)
+			(type solid)
+		)
+		(fill
+			(color 255 106 0 1)
+		)
+		(property "Sheetname" "SD card"
+			(at 20.32 142.7984 0)
+			(show_name no)
+			(do_not_autoplace no)
+			(effects
+				(font
+					(size 1.27 1.27)
+				)
+				(justify left bottom)
+			)
+		)
+		(property "Sheetfile" "schematics\\SD_card.kicad_sch"
+			(at 20.32 156.7946 0)
+			(show_name no)
+			(do_not_autoplace no)
+			(effects
+				(font
+					(size 1.27 1.27)
+				)
+				(justify left top)
+			)
+		)
+		(instances
+			(project "flamingo"
+				(path "/817f49eb-0105-475d-aa60-c8a0ced591cc"
+					(page "10")
+				)
+			)

Commit message: starting schematic work
Other:
- sheet Camera: file schematics\camera.kicad_sch -> schematics/camera.kicad_sch
- sheet Core: file schematics\core.kicad_sch -> schematics/core.kicad_sch
- sheet Debug USB: file schematics\usb_debug.kicad_sch -> schematics/usb_debug.kicad_sch
- sheet GPIO: file schematics\GPIO.kicad_sch -> schematics/GPIO.kicad_sch
- sheet Power: file schematics\power.kicad_sch -> schematics/power.kicad_sch
- sheet Power Program USB: file schematics\usb_power_program.kicad_sch -> schematics/usb_power_program.kicad_sch
- sheet SD card: file schematics\SD_card.kicad_sch -> schematics/SD_card.kicad_sch
Changed lines of the file:
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@@
 			)
 		)
-		(property "Sheetfile" "schematics\\camera.kicad_sch"
+		(property "Sheetfile" "schematics/camera.kicad_sch"
 			(at 74.93 80.5946 0)
 			(show_name no)
@@
 			)
 		)
-		(property "Sheetfile" "schematics\\usb_debug.kicad_sch"
+		(property "Sheetfile" "schematics/usb_debug.kicad_sch"
 			(at 20.32 116.1546 0)
 			(show_name no)
@@
 	)
 	(sheet
-		(at 20.32 87.63)
+		(at 20.32 85.09)
 		(size 110.49 11.43)
 		(exclude_from_sim no)
@@
 		)
 		(property "Sheetname" "Power Program USB"
-			(at 20.32 86.9184 0)
-			(show_name no)
-			(do_not_autoplace no)
-			(effects
-				(font
-					(size 1.27 1.27)
-				)
-				(justify left bottom)
-			)
-		)
-		(property "Sheetfile" "schematics\\usb_power_program.kicad_sch"
-			(at 20.32 99.6446 0)
+			(at 20.32 84.3784 0)
+			(show_name no)
+			(do_not_autoplace no)
+			(effects
+				(font
+					(size 1.27 1.27)
+				)
+				(justify left bottom)
+			)
+		)
+		(property "Sheetfile" "schematics/usb_power_program.kicad_sch"
+			(at 20.32 97.1046 0)
 			(show_name no)
 			(do_not_autoplace no)
@@
 			)
 		)
-		(property "Sheetfile" "schematics\\core.kicad_sch"
+		(property "Sheetfile" "schematics/core.kicad_sch"
 			(at 19.05 78.0546 0)
 			(show_name no)
@@
 			)
 		)
-		(property "Sheetfile" "schematics\\GPIO.kicad_sch"
+		(property "Sheetfile" "schematics/GPIO.kicad_sch"
 			(at 97.79 135.2046 0)
 			(show_name no)
@@
 			)
 		)
-		(property "Sheetfile" "schematics\\power.kicad_sch"
+		(property "Sheetfile" "schematics/power.kicad_sch"
 			(at 19.05 43.7646 0)
 			(show_name no)
@@
 			)
 		)
-		(property "Sheetfile" "schematics\\SD_card.kicad_sch"
+		(property "Sheetfile" "schematics/SD_card.kicad_sch"
 			(at 20.32 156.7946 0)
 			(show_name no)
