File: Flamingo/schematics/core.kicad_sch (KiCad schematic)
At the start: 0 parts

Commit message: starting schematic work
Parts:
- added U?: ESP32-S3-WROOM-1-N16R8, RF_Module:ESP32-S3-WROOM-1, symbol RF_Module:ESP32-S3-WROOM-1
Connections:
- new net: U?.1 (GND), U?.40 (GND), U?.41 (GND)
Changed lines of the file:
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@@
 		(comment 1 "Designed by Simon Kaplinsky ")
 	)
+	(symbol
+		(lib_id "RF_Module:ESP32-S3-WROOM-1")
+		(at 99.06 60.96 0)
+		(unit 1)
+		(body_style 1)
+		(exclude_from_sim no)
+		(in_bom yes)
+		(on_board yes)
+		(in_pos_files yes)
+		(dnp no)
+		(fields_autoplaced yes)
+		(property "Reference" "U?"
+			(at 101.2033 30.48 0)
+			(show_name no)
+			(do_not_autoplace no)
+			(effects
+				(font
+					(size 1.27 1.27)
+				)
+				(justify left)
+			)
+		)
+		(property "Value" "ESP32-S3-WROOM-1-N16R8"
+			(at 101.2033 33.02 0)
+			(show_name no)
+			(do_not_autoplace no)
+			(effects
+				(font
+					(size 1.27 1.27)
+				)
+				(justify left)
+			)
+		)
+		(property "Footprint" "RF_Module:ESP32-S3-WROOM-1"
+			(at 99.06 58.42 0)
+			(hide yes)
+			(show_name no)
+			(do_not_autoplace no)
+			(effects
+				(font
+					(size 1.27 1.27)
+				)
+			)
+		)
+		(property "Datasheet" "https://www.espressif.com/sites/default/files/documentation/esp32-s3-wroom-1_wroom-1u_datasheet_en.pdf"
+			(at 99.06 60.96 0)
+			(hide yes)
+			(show_name no)
+			(do_not_autoplace no)
+			(effects
+				(font
+					(size 1.27 1.27)
+				)
+			)
+		)
+		(property "Description" "RF Module, ESP32-S3 SoC, Wi-Fi 802.11b/g/n, Bluetooth, BLE, 32-bit, 3.3V, onboard antenna, SMD"
+			(at 99.06 60.96 0)
+			(hide yes)
+			(show_name no)
+			(do_not_autoplace no)
+			(effects
+				(font
+					(size 1.27 1.27)
+				)
+			)
+		)
+		(pin "5"
+		)
+		(pin "20"
+		)
+		(pin "10"
+		)
+		(pin "16"
+		)
+		(pin "23"
+		)
+		(pin "21"
+		)
+		(pin "2"
+		)
+		(pin "15"
+		)
+		(pin "30"
+		)
+		(pin "3"
+		)
+		(pin "7"
+		)
+		(pin "8"
+		)
+		(pin "27"
+		)
+		(pin "13"
+		)
+		(pin "14"
+		)
+		(pin "22"
+		)
+		(pin "11"
+		)
+		(pin "17"
+		)
+		(pin "6"
+		)
+		(pin "12"
+		)
+		(pin "4"
+		)
+		(pin "9"
+		)
+		(pin "1"
+		)
+		(pin "18"
+		)
+		(pin "19"
+		)
+		(pin "24"
+		)
+		(pin "25"
+		)
+		(pin "26"
+		)
+		(pin "28"
+		)
+		(pin "29"
+		)
+		(pin "35"
+		)
+		(pin "41"
+		)
+		(pin "40"
+		)
+		(pin "31"
+		)
+		(pin "33"
+		)
+		(pin "38"
+		)
+		(pin "39"
+		)
+		(pin "32"
+		)
+		(pin "34"
+		)
+		(pin "36"
+		)
+		(pin "37"
+		)
+		(instances
+			(project "flamingo"
+				(path "/817f49eb-0105-475d-aa60-c8a0ced591cc/91741965-6759-4532-86dd-7c4d063ae6ad"
+					(reference "U?")
+					(unit 1)
+				)
+			)
+		)
+	)
 )
